File: rgb_sw.kicad_sch (KiCad schematic)
At the start: 13 parts, among them J1 POWER, J2 RGB_TAPE, Q1 IRFZ44N, Q2 IRFZ44N, Q3 IRFZ44N

Commit message: actualizando a kicad 8
Parts:
- H2, H3: now left out of the parts list
Connections:
- net B: now also R3.2; no longer R3.1
- net G: now also R1.2; no longer R1.1
- net at C2.1, Q2.1 (G): now also R1.1; no longer R1.2
- net at C1.1, Q1.1 (G): now also R3.1; no longer R3.2
Other:
- moved on the sheet: C1, C2, C3, J1, J2, Q1, Q2, Q3, R1, R2, R3
